File: PCB/Rev1.1.brd (EAGLE design)
At the start: 101.6 x 81.3 mm, 27 parts, among them U1 ATMEGA328P-PU, U2 BT, U3 SMD_H-BRIDGE

Commit message: Moved ground pour to top copper to get rid of many vias needed for the SMD components.
Routing:
- net GND: track 105.9 -> 1.33 mm, vias 15 -> 0
- net 5V: track 153.7 -> 151.6 mm
- net N$2: track 105.2 -> 106.4 mm
- added copper zone on layer 1, net GND
- removed copper zone on layer 16, net GND
Changed lines of the file:
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@@
 <wire x1="55.88" y1="63.5" x2="91.44" y2="63.5" width="0.4064" layer="21"/>
 <wire x1="91.44" y1="63.5" x2="91.44" y2="17.78" width="0.4064" layer="21"/>
-<wire x1="91.44" y1="17.78" x2="55.88" y2="17.78" width="0.4064" layer="21"/>
 <text x="49.53" y="57.15" size="1.27" layer="25" align="center-right">5V</text>
 <text x="49.53" y="54.61" size="1.27" layer="25" align="center-right">GND</text>
@@
 <text x="30.48" y="76.2" size="0.6096" layer="25" align="center-left">GND</text>
 <text x="22.86" y="76.2" size="0.6096" layer="25" align="center-right">5V</text>
-<text x="96.52" y="67.31" size="2.54" layer="25" rot="R90" align="center">BayouBot v1.1
+<text x="96.52" y="64.77" size="2.54" layer="25" rot="R90" align="center">BayouBot v1.1
 LSU RRL</text>
 <text x="74.93" y="41.91" size="2.54" layer="25" rot="R180" align="center">Place
 Breadboard
 Here</text>
+<wire x1="55.88" y1="17.78" x2="91.44" y2="17.78" width="0.4064" layer="21"/>
 </plain>
 <attributes>
@@
 <contactref element="PROG" pad="6"/>
 <contactref element="LED2" pad="C"/>
-<polygon width="0.4064" layer="16">
+<wire x1="45.72" y1="65.14" x2="45.72" y2="64.99" width="0.4064" layer="1"/>
+<wire x1="13.74" y1="5.08" x2="13.18" y2="5.08" width="0.4064" layer="1"/>
+<wire x1="69.465" y1="75.935" x2="68.845" y2="75.935" width="0.4064" layer="1"/>
+<polygon width="0.4064" layer="1">
 <vertex x="2.54" y="71.12"/>
 <vertex x="10.16" y="71.12"/>
 <vertex x="10.16" y="78.74"/>
-<vertex x="91.44" y="78.74"/>
-<vertex x="91.44" y="2.54"/>
+<vertex x="99.06" y="78.74"/>
+<vertex x="99.06" y="2.54"/>
 <vertex x="10.16" y="2.54"/>
-<vertex x="10.16" y="10.16"/>
-<vertex x="2.54" y="10.16"/>
+<vertex x="10.16" y="8.89"/>
+<vertex x="2.54" y="8.89"/>
 </polygon>
-<wire x1="24.2" y1="59.69" x2="21.59" y2="59.69" width="0.4064" layer="1"/>
-<via x="21.59" y="59.69" extent="1-16" drill="0.6" diameter="0.6096"/>
-<wire x1="21.59" y1="59.69" x2="20.32" y2="59.69" width="0.4064" layer="16"/>
-<wire x1="39.44" y1="71.12" x2="36.83" y2="71.12" width="0.4064" layer="1"/>
-<via x="36.83" y="71.12" extent="1-16" drill="0.6" diameter="0.6096"/>
-<wire x1="36.83" y1="71.12" x2="35.56" y2="71.12" width="0.4064" layer="16"/>
-<wire x1="56.78" y1="74.56" x2="57.15" y2="74.93" width="0.4064" layer="1"/>
-<wire x1="57.15" y1="74.93" x2="58.2" y2="74.93" width="0.4064" layer="1"/>
-<wire x1="58.2" y1="74.93" x2="58.42" y2="74.71" width="0.4064" layer="1"/>
-<wire x1="45.72" y1="65.14" x2="45.72" y2="64.99" width="0.4064" layer="1"/>
-<wire x1="45.72" y1="74.56" x2="51.7" y2="74.56" width="0.4064" layer="1"/>
-<wire x1="51.7" y1="74.56" x2="52.07" y2="74.93" width="0.4064" layer="1"/>
-<via x="52.07" y="74.93" extent="1-16" drill="0.6" diameter="0.6096"/>
-<wire x1="52.07" y1="74.93" x2="52.07" y2="76.2" width="0.4064" layer="16"/>
-<wire x1="43.18" y1="12.48" x2="44.67" y2="12.48" width="0.4064" layer="1"/>
-<wire x1="44.67" y1="12.48" x2="45.72" y2="11.43" width="0.4064" layer="1"/>
-<via x="45.72" y="11.43" extent="1-16" drill="0.6" diameter="0.6096"/>
-<wire x1="45.72" y1="11.43" x2="46.99" y2="11.43" width="0.4064" layer="16"/>
-<wire x1="33.02" y1="39.74" x2="36.46" y2="39.74" width="0.4064" layer="1"/>
-<wire x1="36.46" y1="39.74" x2="36.83" y2="39.37" width="0.4064" layer="1"/>
-<wire x1="16.51" y1="26.6" x2="16.51" y2="27.94" width="0.4064" layer="1"/>
-<via x="16.51" y="27.94" extent="1-16" drill="0.6" diameter="0.6096"/>
-<wire x1="16.51" y1="27.94" x2="7.62" y2="27.94" width="0.4064" layer="16"/>
-<wire x1="13.74" y1="17.78" x2="13.22" y2="17.78" width="0.4064" layer="1"/>
-<wire x1="13.22" y1="17.78" x2="12.1" y2="16.66" width="0.4064" layer="1"/>
-<wire x1="13.74" y1="5.08" x2="13.18" y2="5.08" width="0.4064" layer="1"/>
-<wire x1="13.18" y1="5.08" x2="12.1" y2="6.16" width="0.4064" layer="1"/>
-<wire x1="13.74" y1="17.78" x2="13.74" y2="5.08" width="0.4064" layer="1"/>
-<wire x1="13.74" y1="17.78" x2="13.74" y2="18.01" width="0.4064" layer="1"/>
-<wire x1="13.74" y1="18.01" x2="11.43" y2="20.32" width="0.4064" layer="1"/>
-<via x="11.43" y="20.32" extent="1-16" drill="0.6" diameter="0.6096"/>
-<wire x1="11.43" y1="20.32" x2="11.43" y2="21.59" width="0.4064" layer="16"/>
-<wire x1="41.69" y1="62.23" x2="43.18" y2="62.23" width="0.4064" layer="1"/>
-<wire x1="29.21" y1="63.13" x2="30.11" y2="63.13" width="0.4064" layer="1"/>
-<wire x1="30.11" y1="63.13" x2="31.75" y2="64.77" width="0.4064" layer="1"/>
-<via x="31.75" y="64.77" extent="1-16" drill="0.6" diameter="0.6096"/>
-<wire x1="31.75" y1="64.77" x2="31.75" y2="66.04" width="0.4064" layer="16"/>
-<wire x1="69.465" y1="75.935" x2="68.845" y2="75.935" width="0.4064" layer="1"/>
-<wire x1="68.845" y1="75.935" x2="67.31" y2="77.47" width="0.4064" layer="1"/>
-<via x="67.31" y="77.47" extent="1-16" drill="0.6" diameter="0.6096"/>
-<wire x1="67.31" y1="77.47" x2="68.58" y2="77.47" width="0.4064" layer="16"/>
-<wire x1="75.315" y1="71.385" x2="75.315" y2="70.235" width="0.4064" layer="1"/>
-<wire x1="75.315" y1="70.235" x2="74.93" y2="69.85" width="0.4064" layer="1"/>
-<via x="74.93" y="69.85" extent="1-16" drill="0.6" diameter="0.6096"/>
-<wire x1="74.93" y1="69.85" x2="73.66" y2="69.85" width="0.4064" layer="16"/>
-<wire x1="79.64" y1="77.47" x2="81.28" y2="77.47" width="0.4064" layer="1"/>
-<via x="81.28" y="77.47" extent="1-16" drill="0.6" diameter="0.6096"/>
-<wire x1="81.28" y1="77.47" x2="82.55" y2="77.47" width="0.4064" layer="16"/>
-<wire x1="43.18" y1="62.23" x2="44.45" y2="63.5" width="0.4064" layer="1"/>
-<via x="44.45" y="63.5" extent="1-16" drill="0.6" diameter="0.6096"/>
-<wire x1="44.45" y1="63.5" x2="45.72" y2="63.5" width="0.4064" layer="16"/>
-<wire x1="45.72" y1="65.14" x2="45.72" y2="64.77" width="0.4064" layer="1"/>
-<wire x1="45.72" y1="64.77" x2="44.45" y2="63.5" width="0.4064" layer="1"/>
-<wire x1="21.22" y1="24.13" x2="21.22" y2="22.49" width="0.4064" layer="1"/>
-<wire x1="21.22" y1="22.49" x2="20.32" y2="21.59" width="0.4064" layer="1"/>
-<via x="20.32" y="21.59" extent="1-16" drill="0.6" diameter="0.6096"/>
-<wire x1="20.32" y1="21.59" x2="21.59" y2="21.59" width="0.4064" layer="16"/>
-<wire x1="17.41" y1="21.59" x2="20.32" y2="21.59" width="0.4064" layer="1"/>
-<wire x1="28.31" y1="21.59" x2="24.13" y2="21.59" width="0.4064" layer="1"/>
-<via x="24.13" y="21.59" extent="1-16" drill="0.6" diameter="0.6096"/>
-<wire x1="24.13" y1="21.59" x2="22.86" y2="21.59" width="0.4064" layer="16"/>
-<wire x1="58.42" y1="6.57" x2="62.01" y2="6.57" width="0.8128" layer="1"/>
-<wire x1="62.01" y1="6.57" x2="62.23" y2="6.35" width="0.8128" layer="1"/>
-<via x="62.23" y="6.35" extent="1-16" drill="0.6" diameter="0.6096"/>
-<wire x1="62.23" y1="6.35" x2="63.5" y2="6.35" width="0.8128" layer="16"/>
-<wire x1="56.78" y1="74.56" x2="52.44" y2="74.56" width="0.8128" layer="1"/>
-<wire x1="52.44" y1="74.56" x2="52.07" y2="74.93" width="0.8128" layer="1"/>
-<wire x1="71.12" y1="67.68" x2="71.12" y2="67.31" width="0.4064" layer="1"/>
-<wire x1="71.12" y1="67.31" x2="68.58" y2="66.04" width="0.4064" layer="1"/>
-<via x="68.58" y="66.04" extent="1-16" drill="0.6" diameter="0.6096"/>
-<wire x1="68.58" y1="66.04" x2="69.85" y2="66.04" width="0.4064" layer="16"/>
 </signal>
 <signal name="N$1" class="1">
@@
 <wire x1="35.24" y1="72.07" x2="33.02" y2="69.85" width="0.4064" layer="1"/>
 <wire x1="23.88" y1="60.96" x2="24.2" y2="60.64" width="0.4064" layer="1"/>
-<wire x1="15.56" y1="26.6" x2="15.56" y2="29.53" width="0.4064" layer="1"/>
-<wire x1="15.56" y1="29.53" x2="17.46" y2="31.43" width="0.4064" layer="1"/>
-<wire x1="17.46" y1="26.6" x2="17.46" y2="31.43" width="0.4064" layer="1"/>
 <wire x1="17.15" y1="64.23" x2="17.15" y2="64.13" width="0.4064" layer="1"/>
 <wire x1="17.15" y1="64.13" x2="20.32" y2="60.96" width="0.4064" layer="1"/>
@@
 <wire x1="24.2" y1="58.74" x2="20.635" y2="58.74" width="0.4064" layer="1"/>
 <wire x1="20.635" y1="58.74" x2="20.32" y2="59.055" width="0.4064" layer="1"/>
-<wire x1="17.46" y1="31.43" x2="17.46" y2="46.04" width="0.4064" layer="1"/>
-<wire x1="17.46" y1="46.04" x2="5.08" y2="58.42" width="0.4064" layer="1"/>
-<wire x1="5.08" y1="58.42" x2="5.08" y2="61.06" width="0.4064" layer="1"/>
-<wire x1="5.08" y1="61.06" x2="8.25" y2="64.23" width="0.4064" layer="1"/>
+<wire x1="15.56" y1="26.6" x2="15.56" y2="30.16" width="0.4064" layer="1"/>
+<wire x1="15.56" y1="30.16" x2="15.24" y2="30.48" width="0.4064" layer="1"/>
+<wire x1="15.24" y1="30.48" x2="11.43" y2="30.48" width="0.4064" layer="1"/>
+<wire x1="11.43" y1="30.48" x2="3.81" y2="38.1" width="0.4064" layer="1"/>
+<wire x1="3.81" y1="38.1" x2="3.81" y2="59.79" width="0.4064" layer="1"/>
+<wire x1="3.81" y1="59.79" x2="8.25" y2="64.23" width="0.4064" layer="1"/>
+<wire x1="17.46" y1="26.6" x2="17.46" y2="28.26" width="0.4064" layer="1"/>
+<wire x1="17.46" y1="28.26" x2="15.56" y2="30.16" width="0.4064" layer="1"/>
 </signal>
 <signal name="5V" class="1">
@@
 <wire x1="77.47" y1="77.47" x2="76.2" y2="78.74" width="0.4064" layer="1"/>
 <wire x1="76.2" y1="78.74" x2="44.45" y2="78.74" width="0.4064" layer="1"/>
-<wire x1="44.45" y1="78.74" x2="40.64" y2="74.93" width="0.4064" layer="1"/>
-<via x="40.64" y="74.93" extent="1-16" drill="0.6" diameter="0.6096"/>
-<wire x1="40.64" y1="74.93" x2="40.64" y2="71.12" width="0.4064" layer="16"/>
-<wire x1="40.64" y1="71.12" x2="43.18" y2="68.58" width="0.4064" layer="16"/>
-<wire x1="43.18" y1="68.58" x2="43.18" y2="59.69" width="0.4064" layer="16"/>
 <wire x1="77.47" y1="77.47" x2="76.85" y2="77.47" width="0.4064" layer="1"/>
 <wire x1="76.85" y1="77.47" x2="75.315" y2="75.935" width="0.4064" layer="1"/>
 <wire x1="44.45" y1="39.37" x2="44.45" y2="36.83" width="0.4064" layer="1"/>
+<wire x1="44.45" y1="78.74" x2="43.18" y2="77.47" width="0.4064" layer="1"/>
+<via x="43.18" y="77.47" extent="1-16" drill="0.6" diameter="0.6096"/>
+<wire x1="43.18" y1="77.47" x2="43.18" y2="59.69" width="0.4064" layer="16"/>
 <wire x1="29.21" y1="60.96" x2="29.21" y2="61.33" width="0" layer="19" extent="1-1"/>
 </signal>
